File: PCB/pcb/pcb.kicad_pcb (KiCad board)
At the start: 2 copper layers, 148 parts, among them J1 USB_B_Micro, SW1 SW_Push, U1 ATmega32U4-AU, Y1 16MHz

Commit message: Layout the switches and diodes
Parts:
- removed the D2 at (213.9, 401.2)
- removed the D53 at (336.1, 405.8)
- removed the D58 at (341.6, 402.5)
- removed the MX18 at (111.2, 142.4)
- removed the MX33 at (179.0, 61.0)
- removed SW1: SW_Push, Button_Switch_SMD:SW_SPST_B3S-1000
- added D14: 1N4148W, Diode_SMD:D_SOD-123, B.Cu at (281.9, 33.3)
- added D15: 1N4148W, Diode_SMD:D_SOD-123, B.Cu at (301.0, 33.3)
- added D16: 1N4148W, Diode_SMD:D_SOD-123, B.Cu at (38.7, 52.1)
- added JP1: Jumper_NO_Small, Jumper:SolderJumper-2_P1.3mm_Open_RoundedPad1.0x1.5mm, F.Cu at (45.2, 169.1)
- added MX34: D, MX_Only:MXOnly-1U-NoLED, F.Cu at (97.6, 66.7)
- added MX9: 8, MX_Only:MXOnly-1U-NoLED, F.Cu at (178.6, 28.6)
- C1: renamed from C4; value 0.1u -> 1u
- C2: renamed from C7; value 0.1u -> 100n
- C3: renamed from C8; value 0.1u -> 100n
- C4: renamed from C9; value 0.1u -> 100n
- C5: renamed from C10; value 4.7u -> 100n
- MX61: renamed from MX32; footprint MX_Only:MXOnly-7U-ReversedStabilizers -> MX_Only:MXOnly-7U-ReversedStabilizers-NoLED
- Y1: footprint Crystal:Crystal_SMD_5032-2Pin_5.0x3.2mm_HandSoldering -> Crystal:Crystal_SMD_5032-4Pin_5.0x3.2mm; moved to F.Cu
- moved D1 458.4 mm to (34.3, 33.3), turned to 90 degrees
- moved D31 428.5 mm to (41.9, 71.1), turned to 90 degrees
- moved D3 427.8 mm to (72.4, 33.3), turned to 90 degrees
- moved U1 415.4 mm to (58.4, 104.1), turned to 45 degrees
- moved D2 412.8 mm to (53.3, 33.3), turned to 90 degrees
- moved D45 408.6 mm to (45.1, 90.2), turned to 90 degrees
- moved D4 399.5 mm to (91.4, 33.3), turned to 90 degrees
- moved D5 397.1 mm to (110.5, 33.3), turned to 90 degrees
- moved D36 390.6 mm to (144.1, 71.1), turned to 90 degrees
- moved D17 388.8 mm to (62.9, 52.1), turned to 90 degrees
- moved D18 385.8 mm to (81.9, 52.1), turned to 90 degrees
- moved D9 384.5 mm to (186.7, 33.3), turned to 90 degrees
- moved D32 383.5 mm to (67.9, 71.1), turned to 90 degrees
- moved D10 381.3 mm to (205.7, 33.3), turned to 90 degrees
- moved D8 380.2 mm to (167.6, 33.3), turned to 90 degrees
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- renumbered C5 to C6, C6 to C7, C2 to C8, C1 to C9, D37 to D10, D41 to D11, D45 to D12, D50 to D13, D8 to D17, D12 to D18, D17 to D19, D5 to D2, D21 to D20, D25 to D21, D29 to D22, D34 to D23, D38 to D24, D42 to D25, D46 to D26, D51 to D27, D54 to D28, D59 to D29, D7 to D3, D62 to D30, D3 to D31, D9 to D32, D13 to D33, D18 to D34, D22 to D35, D26 to D36, D30 to D37, D35 to D38, D11 to D4, D43 to D40, D47 to D41, D52 to D42, D55 to D43, D63 to D44, D6 to D45, D10 to D46, D14 to D47, D19 to D48, D23 to D49, D16 to D5, D27 to D50, D31 to D51, D36 to D52, D40 to D53, D44 to D54, D48 to D55, D60 to D57, D64 to D58, D4 to D59, D20 to D6, D15 to D60, D32 to D61, D49 to D62, D57 to D63, D61 to D64, D24 to D7, D28 to D8, D33 to D9, MX37 to MX10, MX41 to MX11, MX45 to MX12, MX50 to MX13, MX53 to MX14, MX58 to MX15, MX2 to MX16, MX8 to MX17, MX12 to MX18, MX17 to MX19, MX5 to MX2, MX21 to MX20, MX25 to MX21, MX29 to MX22, MX34 to MX23, MX38 to MX24, MX42 to MX25, MX46 to MX26, MX51 to MX27, MX54 to MX28, MX59 to MX29, MX7 to MX3, MX62 to MX30, MX3 to MX31, MX9 to MX32, MX13 to MX33, MX22 to MX35, MX26 to MX36, MX30 to MX37, MX35 to MX38, MX11 to MX4, MX43 to MX40, MX47 to MX41, MX52 to MX42, MX55 to MX43, MX63 to MX44, MX6 to MX45, MX10 to MX46, MX14 to MX47, MX19 to MX48, MX23 to MX49, MX16 to MX5, MX27 to MX50, MX31 to MX51, MX36 to MX52, MX40 to MX53, MX44 to MX54, MX48 to MX55, MX60 to MX57, MX64 to MX58, MX4 to MX59, MX20 to MX6, MX15 to MX60, MX49 to MX62, MX57 to MX63, MX61 to MX64, MX24 to MX7, MX28 to MX8, R3 to R1, R4 to R2, R5 to R3, R2 to R4, R1 to R5
Connections:
- J1 pad 4: Net-(J1-Pad4) -> (no net)
- U1 pad 1: Net-(U1-Pad1) -> (no net)
- U1 pad 10: row2 -> col2
- U1 pad 11: row3 -> col3
- U1 pad 12: col2 -> (no net)
- U1 pad 18: col5 -> row4
- U1 pad 19: col6 -> row0
- U1 pad 20: col7 -> row1
- U1 pad 21: col8 -> row2
- U1 pad 22: col10 -> row3
- U1 pad 25: col9 -> (no net)
- U1 pad 26: col11 -> (no net)
- U1 pad 27: col12 -> col15
- U1 pad 28: row4 -> col14
- U1 pad 29: col0 -> col13
- U1 pad 30: col1 -> col12
- U1 pad 31: col3 -> col11
- U1 pad 32: col4 -> col10
- U1 pad 36: Net-(U1-Pad36) -> col9
- U1 pad 37: Net-(U1-Pad37) -> col8
- U1 pad 38: Net-(U1-Pad38) -> col7
- U1 pad 39: col15 -> col6
- U1 pad 40: col14 -> col5
- U1 pad 41: col13 -> col4
- U1 pad 42: Net-(U1-Pad42) -> (no net)
- U1 pad 8: row0 -> col0
- U1 pad 9: row1 -> col1
- Y1 pad 2: XTAL2 -> GND
Other:
- board outline added: 309.6 x 100 mm
- net class Default: clearance 0.2 -> 0.127
- rule trace_clearance: 0.2 -> 0.127

Commit message: Route the matrix
Routing:
- net row1: track 0.00 -> 371.3 mm
- net row0: track 0.00 -> 369.2 mm
- net row2: track 0.00 -> 336.1 mm
- net row4: track 0.00 -> 315.0 mm
- net row3: track 0.00 -> 292.3 mm
- net col13: track 0.00 -> 107.7 mm
- net col3: track 0.00 -> 91.9 mm
- net col14: track 0.00 -> 91.0 mm
- net col11: track 0.00 -> 87.9 mm
- net col0: track 0.00 -> 82.7 mm
- net col9: track 0.00 -> 67.9 mm
- net col8: track 0.00 -> 67.9 mm
- net col2: track 0.00 -> 67.9 mm
- net col10: track 0.00 -> 67.9 mm
- net col7: track 0.00 -> 67.9 mm
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
Commit message: Layout the PCB and generate Gerbers.
I am an idiot. This is my first pass at laying out the board.

What I should have done is mark out the edge cuts and then generate a 3d
model to import into Fusion to check that it fits in the case.

I did not do this until after I'd layed out the board :'( and it's about
5mm too long on each side.

So now I need to make the board smaller by a significant amount and redo
the layout.

Think I learned a lot about laying out a PCB though.
Parts:
- JP1, Y1: moved to B.Cu
- moved R3 258.6 mm to (35.3, 24.9), turned to 270 degrees
- moved J1 240.6 mm to (36.8, 19.3), turned to 0 degrees
- moved R2 225.9 mm to (38.1, 24.9), turned to 90 degrees
- moved C4 219.3 mm to (119.9, 100.1), turned to 270 degrees
- moved C3 215.2 mm to (117.1, 100.1), turned to 270 degrees
- moved C2 211.2 mm to (114.3, 100.1), turned to 270 degrees
- moved R1 211.0 mm to (147.1, 104.1), turned to 90 degrees
- moved C1 210.2 mm to (122.7, 100.1), turned to 270 degrees
- moved C7 205.1 mm to (120.9, 111.3), turned to 0 degrees
- moved C6 201.7 mm to (115.6, 108.0), turned to 270 degrees
- moved C5 201.1 mm to (143.0, 109.5), turned to 90 degrees
- moved R4 196.0 mm to (129.5, 114.8)
- moved C8 192.5 mm to (135.4, 114.6), turned to 0 degrees
- moved R5 190.0 mm to (115.1, 113.8)
- moved C9 189.7 mm to (124.7, 113.8), turned to 0 degrees
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Connections:
- U1 pad 10: col2 -> col1
- U1 pad 11: col3 -> col0
- U1 pad 27: col15 -> col10
- U1 pad 28: col14 -> col11
- U1 pad 29: col13 -> col12
- U1 pad 30: col12 -> col13
- U1 pad 31: col11 -> col14
- U1 pad 32: col10 -> col15
- U1 pad 8: col0 -> col3
- U1 pad 9: col1 -> col2
Routing:
- net USB_VBUS: track 0.00 -> 233.1 mm, vias 0 -> 7
- net GND: track 0.00 -> 227.3 mm, vias 0 -> 6
- net USB_Dneg: track 0.00 -> 197.4 mm, vias 0 -> 2
- net USB_Dpos: track 0.00 -> 190.3 mm, vias 0 -> 2
- net col15: track 64.5 -> 251.4 mm, vias 0 -> 1
- net col14: track 91.0 -> 261.4 mm, vias 0 -> 1
- net col12: track 45.0 -> 200.8 mm, vias 0 -> 1
- net col13: track 107.7 -> 256.9 mm, vias 0 -> 1
- net col1: track 61.1 -> 171.8 mm, vias 0 -> 1
- net col11: track 87.9 -> 197.8 mm, vias 0 -> 1
- net col0: track 82.7 -> 188.0 mm, vias 0 -> 1
- net col10: track 67.9 -> 166.3 mm, vias 0 -> 1
- net col2: track 67.9 -> 155.0 mm, vias 0 -> 1
- net col9: track 67.9 -> 143.5 mm, vias 0 -> 3
- net row0: track 369.2 -> 443.0 mm
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- added copper zone on B.Cu, net GND
