File: PCB/pcb/pcb.kicad_pcb (KiCad board)
At the start: 2 copper layers, 309.6 x 100 mm, 147 parts, among them J1 USB_B_Micro, U1 ATmega32U4-AU, Y1 16MHz

Commit message: Layout and generate gerbers
The board is too big
Parts:
- added MX53: LANGLE, MX_Only:MXOnly-1U-NoLED, F.Cu at (202.4, 85.7)
Routing:
- net GND: track 33.2 -> 227.3 mm, vias 0 -> 6
- net USB_VBUS: track 82.6 -> 233.1 mm, vias 4 -> 7
- net col10: track 96.7 -> 166.3 mm
- net col15: track 184.7 -> 251.4 mm
- net col14: track 258.0 -> 261.4 mm
- net col13: track 254.8 -> 256.9 mm
- net col12: track 199.2 -> 200.8 mm
- net col11: track 196.8 -> 197.8 mm
