File: PCB/pcb/pcb.kicad_pcb (KiCad board)
At the start: 2 copper layers, 148 parts, among them J1 USB_B_Micro, U1 ATmega32U4-AU, Y1 16MHz

Commit message: WIP
Parts:
- moved J1 275.1 mm to (311.9, 21.7)
- moved D1 8.19 mm to (34.3, 25.1)
- moved D10 8.19 mm to (205.7, 25.1)
- moved D11 8.19 mm to (224.8, 25.1)
- moved D12 8.19 mm to (243.8, 25.1)
- moved D13 8.19 mm to (262.9, 25.1)
- moved D14 8.19 mm to (281.9, 25.1)
- moved D15 8.19 mm to (301.0, 25.1)
- moved D2 8.19 mm to (53.3, 25.1)
- moved D3 8.19 mm to (72.4, 25.1)
- moved D4 8.19 mm to (91.4, 25.1)
- moved D5 8.19 mm to (110.5, 25.1)
- moved D6 8.19 mm to (129.5, 25.1)
- moved D7 8.19 mm to (148.6, 25.1)
- moved D8 8.19 mm to (167.6, 25.1)
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Routing:
- net row0: track 0.00 -> 444.9 mm
- net Net-(D15-Pad2): track 0.00 -> 5.56 mm
- net Net-(D9-Pad2): track 0.00 -> 5.56 mm
- net Net-(D7-Pad2): track 0.00 -> 5.56 mm
- net Net-(D3-Pad2): track 0.00 -> 5.56 mm
- net Net-(D2-Pad2): track 0.00 -> 5.56 mm
- net Net-(D12-Pad2): track 0.00 -> 5.56 mm
- net Net-(D11-Pad2): track 0.00 -> 5.56 mm
- net Net-(D10-Pad2): track 0.00 -> 5.56 mm
- net Net-(D1-Pad2): track 0.00 -> 5.56 mm
- net Net-(D5-Pad2): track 0.00 -> 5.56 mm
- net Net-(D6-Pad2): track 0.00 -> 5.56 mm
- net Net-(D4-Pad2): track 0.00 -> 5.56 mm
- net Net-(D8-Pad2): track 0.00 -> 5.56 mm
- net Net-(D14-Pad2): track 0.00 -> 5.56 mm
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Other:
- board outline added: 304.8 x 95.3 mm

Commit message: Layout components around MC
Move diodes to be differently oriented
Parts:
- moved R2 271.9 mm to (314.5, 31.8)
- moved R3 271.2 mm to (310.9, 31.8)
- moved C2 86.9 mm to (201.9, 106.9), turned to 90 degrees
- moved C3 84.3 mm to (202.7, 99.6)
- moved C1 72.8 mm to (195.1, 112.8), turned to 180 degrees
- moved C4 69.4 mm to (190.5, 93.5), turned to 180 degrees
- moved C6 64.3 mm to (180.8, 98.6), turned to 180 degrees
- moved U1 58.9 mm to (193.0, 102.1)
- moved C7 58.7 mm to (180.8, 107.7)
- moved Y1 58.4 mm to (180.8, 102.9)
- moved R1 57.8 mm to (204.2, 95.8), turned to 180 degrees
- moved R5 54.0 mm to (170.2, 106.7), turned to 270 degrees
- moved C9 48.8 mm to (174.8, 108.0)
- moved C8 44.9 mm to (190.8, 112.8), turned to 180 degrees
- moved C5 42.3 mm to (186.2, 112.8), turned to 0 degrees
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Routing:
- net row0: track 444.9 -> 0.00 mm
- net Net-(D15-Pad2): track 5.56 -> 0.00 mm
- net Net-(D9-Pad2): track 5.56 -> 0.00 mm
- net Net-(D7-Pad2): track 5.56 -> 0.00 mm
- net Net-(D3-Pad2): track 5.56 -> 0.00 mm
- net Net-(D2-Pad2): track 5.56 -> 0.00 mm
- net Net-(D12-Pad2): track 5.56 -> 0.00 mm
- net Net-(D11-Pad2): track 5.56 -> 0.00 mm
- net Net-(D10-Pad2): track 5.56 -> 0.00 mm
- net Net-(D1-Pad2): track 5.56 -> 0.00 mm
- net Net-(D5-Pad2): track 5.56 -> 0.00 mm
- net Net-(D6-Pad2): track 5.56 -> 0.00 mm
- net Net-(D4-Pad2): track 5.56 -> 0.00 mm
- net Net-(D8-Pad2): track 5.56 -> 0.00 mm
- net Net-(D14-Pad2): track 5.56 -> 0.00 mm
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- added copper zone on B.Cu, net GND

Commit message: Finish Layout
Parts:
- moved C5 19.4 mm to (204.7, 106.9), turned to 90 degrees
- moved C1 16.7 mm to (205.2, 99.6), turned to 270 degrees
- moved C6 3.07 mm to (178.1, 97.3)
- moved Y1 3.07 mm to (178.1, 101.6)
- moved C8 2.17 mm to (192.8, 112.0), turned to 0 degrees
- moved C7 1.08 mm to (180.1, 106.9)
- moved R4 1.02 mm to (172.2, 111.8)
- moved D10 0.25 mm to (197.9, 33.5)
- moved D12 0.25 mm to (236.0, 33.5)
- moved D29 0.25 mm to (288.3, 52.6)
- moved D30 0.25 mm to (312.2, 52.6)
- moved D43 0.25 mm to (281.2, 71.6)
- moved D44 0.25 mm to (312.2, 71.6)
- moved D51 0.25 mm to (164.6, 90.7)
- moved D53 0.25 mm to (202.7, 90.7)
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Connections:
- U1 pad 27: col10 -> col9
- U1 pad 28: col11 -> col10
- U1 pad 29: col12 -> col11
- U1 pad 30: col13 -> col12
- U1 pad 31: col14 -> col13
- U1 pad 32: col15 -> col14
- U1 pad 36: col9 -> col15
Routing:
- net row1: track 0.00 -> 543.1 mm
- net row0: track 0.00 -> 532.3 mm
- net row2: track 0.00 -> 507.2 mm
- net row3: track 0.00 -> 475.7 mm
- net row4: track 0.00 -> 368.3 mm
- net GND: track 0.00 -> 274.4 mm, vias 0 -> 8
- net USB_VBUS: track 0.00 -> 256.7 mm, vias 0 -> 8
- net col0: track 0.00 -> 253.4 mm, vias 0 -> 1
- net col1: track 0.00 -> 232.5 mm, vias 0 -> 1
- net col3: track 0.00 -> 218.7 mm, vias 0 -> 1
- net col2: track 0.00 -> 217.7 mm, vias 0 -> 1
- net USB_Dpos: track 0.00 -> 185.8 mm, vias 0 -> 2
- net col14: track 0.00 -> 182.8 mm, vias 0 -> 1
- net col13: track 0.00 -> 182.4 mm, vias 0 -> 1
- net col4: track 0.00 -> 179.6 mm, vias 0 -> 1
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
Commit message: Move the USB port and regenerate the Gerbers
Parts:
- added J2: ICSP, Connector_PinHeader_2.54mm:PinHeader_2x03_P2.54mm_Vertical, F.Cu at (131.3, 98.6)
- JP1: value Jumper_NO_Small -> RESET; footprint Jumper:SolderJumper-2_P1.3mm_Open_RoundedPad1.0x1.5mm -> Connector_PinSocket_2.54mm:PinSocket_1x02_P2.54mm_Vertical
- R2, R3: value 10k -> 22
- R4: value R_Small -> 10k
- moved R4 12.0 mm to (183.4, 107.4), turned to 270 degrees
- moved J1 9.48 mm to (302.4, 21.7)
- moved R2 7.18 mm to (308.0, 28.6)
- moved R3 6.89 mm to (304.7, 28.6)
- moved C9 2.17 mm to (172.7, 107.2)
- moved R5 1.83 mm to (168.7, 105.7)
- moved C7 1.02 mm to (180.1, 105.9)
- moved JP1 0.76 mm to (173.0, 99.6)
Connections:
- net Net-(C9-Pad1) renamed RESET
- net col0 renamed MISO
- net col1 renamed MOSI
- net col2 renamed SCK
Routing:
- net GND: track 274.4 -> 90.7 mm
- net USB_VBUS: track 256.7 -> 349.8 mm
- net MISO: track 253.4 -> 321.9 mm
- net RESET: track 31.5 -> 85.7 mm, vias 0 -> 1
- net row4: track 368.3 -> 421.2 mm
- net MOSI: track 232.5 -> 255.6 mm, vias 1 -> 2
- net SCK: track 217.7 -> 239.3 mm, vias 1 -> 2
- net USB_Dneg: track 179.4 -> 181.0 mm
- net Net-(J1-Pad2): track 7.25 -> 5.76 mm
- net XTAL2: track 16.0 -> 14.7 mm
- net Net-(JP1-Pad2): track 5.75 -> 6.75 mm
Other:
- rule trace_min: 0.2 -> 0.127
- rule via_min_drill: 0.3 -> 0.2
- rule via_min_size: 0.4 -> 0.45

Commit message: PCB progress
Routing:
- net row4: track 421.2 -> 401.6 mm
- net GND: track 90.7 -> 91.9 mm
- net USB_Dneg: track 181.0 -> 182.1 mm
- net USB_Dpos: track 186.1 -> 186.8 mm
Changed lines of the file:
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@@
   )
   (setup
-    (last_trace_width 0.25)
+    (last_trace_width 0.4064)
     (user_trace_width 0.3048)
     (user_trace_width 0.4064)
@@
   (segment (start 182.804 103.708) (end 187.34 103.708) (width 0.4064) (layer B.Cu) (net 1))
   (segment (start 182.118 104.394) (end 182.804 103.708) (width 0.4064) (layer B.Cu) (net 1))
+  (segment (start 304.32896 23.12748) (end 304.74896 22.70748) (width 0.4064) (layer B.Cu) (net 1))
+  (segment (start 303.72896 23.12748) (end 304.32896 23.12748) (width 0.4064) (layer B.Cu) (net 1))
   (segment (start 200.079 106.108) (end 201.93 107.959) (width 0.6096) (layer B.Cu) (net 2))
   (segment (start 198.74 106.108) (end 200.079 106.108) (width 0.6096) (layer B.Cu) (net 2))
@@
   (segment (start 85.88375 32.86025) (end 85.216 33.528) (width 0.4064) (layer B.Cu) (net 11))
   (segment (start 85.88375 23.495) (end 85.88375 32.86025) (width 0.4064) (layer B.Cu) (net 11))
-  (segment (start 28.7356 109.728) (end 24.671049 105.663449) (width 0.4064) (layer B.Cu) (net 12))
-  (segment (start 28.987753 98.239799) (end 38.826735 98.239799) (width 0.4064) (layer B.Cu) (net 12))
-  (segment (start 24.671049 102.556503) (end 28.987753 98.239799) (width 0.4064) (layer B.Cu) (net 12))
-  (segment (start 24.671049 105.663449) (end 24.671049 102.556503) (width 0.4064) (layer B.Cu) (net 12))
-  (segment (start 38.826735 98.239799) (end 40.231165 99.64423) (width 0.4064) (layer B.Cu) (net 12))
-  (segment (start 29.592 109.728) (end 28.7356 109.728) (width 0.4064) (layer B.Cu) (net 12))
-  (segment (start 40.231165 99.64423) (end 42.418 99.64423) (width 0.4064) (layer B.Cu) (net 12))
-  (segment (start 52.50177 109.728) (end 77.09 109.728) (width 0.4064) (layer B.Cu) (net 12))
-  (segment (start 42.418 99.64423) (end 52.50177 109.728) (width 0.4064) (layer B.Cu) (net 12))
   (segment (start 310.516 110.7344) (end 309.4904 111.76) (width 0.4064) (layer B.Cu) (net 12))
   (segment (start 310.516 109.728) (end 310.516 110.7344) (width 0.4064) (layer B.Cu) (net 12))
@@
   (segment (start 158.116 109.728) (end 102.362 109.728) (width 0.4064) (layer B.Cu) (net 12))
   (segment (start 102.362 109.728) (end 101.681532 109.728) (width 0.4064) (layer B.Cu) (net 12))
+  (segment (start 30.4484 109.728) (end 32.3026 111.5822) (width 0.4064) (layer B.Cu) (net 12))
+  (segment (start 29.592 109.728) (end 30.4484 109.728) (width 0.4064) (layer B.Cu) (net 12))
+  (segment (start 74.6379 111.5822) (end 76.4921 109.728) (width 0.4064) (layer B.Cu) (net 12))
+  (segment (start 32.3026 111.5822) (end 74.6379 111.5822) (width 0.4064) (layer B.Cu) (net 12))
+  (segment (start 76.4921 109.728) (end 77.09 109.728) (width 0.4064) (layer B.Cu) (net 12))
   (segment (start 104.8684 33.528) (end 104.012 33.528) (width 0.4064) (layer B.Cu) (net 13))
   (segment (start 104.93375 33.46265) (end 104.8684 33.528) (width 0.4064) (layer B.Cu) (net 13))
@@
   (segment (start 201.7884 101.6) (end 199.8964 99.708) (width 0.4064) (layer B.Cu) (net 89))
   (segment (start 208.28 101.6) (end 201.7884 101.6) (width 0.4064) (layer B.Cu) (net 89))
-  (segment (start 194.64 110.312) (end 194.64 107.808) (width 0.6096) (layer B.Cu) (net 90))
-  (segment (start 197.23099 112.90299) (end 194.64 110.312) (width 0.6096) (layer B.Cu) (net 90))
-  (segment (start 211.70901 112.90299) (end 197.23099 112.90299) (width 0.6096) (layer B.Cu) (net 90))
-  (segment (start 211.70901 112.90299) (end 212.21701 112.90299) (width 0.6096) (layer B.Cu) (net 90))
-  (via (at 302.26 95.25) (size 0.8) (drill 0.4) (layers F.Cu B.Cu) (net 90))
-  (segment (start 229.87 95.25) (end 302.26 95.25) (width 0.6096) (layer B.Cu) (net 90))
-  (segment (start 212.21701 112.90299) (end 229.87 95.25) (width 0.6096) (layer B.Cu) (net 90))
   (via (at 302.641 35.306) (size 0.8) (drill 0.4) (layers F.Cu B.Cu) (net 90))
-  (segment (start 302.26 35.687) (end 302.641 35.306) (width 0.6096) (layer F.Cu) (net 90))
-  (segment (start 302.26 95.25) (end 302.26 35.687) (width 0.6096) (layer F.Cu) (net 90))
   (segment (start 307.81846 30.12854) (end 307.98516 30.12854) (width 0.6096) (layer B.Cu) (net 90))
   (segment (start 302.641 35.306) (end 307.81846 30.12854) (width 0.6096) (layer B.Cu) (net 90))
+  (segment (start 212.21701 112.90299) (end 227.3808 97.7392) (width 0.6096) (layer B.Cu) (net 90))
+  (segment (start 194.64 110.312) (end 197.23099 112.90299) (width 0.6096) (layer B.Cu) (net 90))
+  (segment (start 197.23099 112.90299) (end 212.21701 112.90299) (width 0.6096) (layer B.Cu) (net 90))
+  (segment (start 194.64 107.808) (end 194.64 110.312) (width 0.6096) (layer B.Cu) (net 90))
+  (segment (start 227.3808 97.7392) (end 231.9782 97.7392) (width 0.6096) (layer B.Cu) (net 90))
+  (segment (start 302.26 96.4819) (end 300.990216 97.751684) (width 0.6096) (layer F.Cu) (net 90))
+  (segment (start 231.9782 97.7392) (end 300.990216 97.751684) (width 0.6096) (layer B.Cu) (net 90))
+  (segment (start 302.26 35.687) (end 302.26 96.4819) (width 0.6096) (layer F.Cu) (net 90))
+  (segment (start 302.641 35.306) (end 302.26 35.687) (width 0.6096) (layer F.Cu) (net 90))
+  (via (at 300.990216 97.751684) (size 0.8) (drill 0.4) (layers F.Cu B.Cu) (net 90))
   (segment (start 197.612 112.014) (end 211.556278 112.014) (width 0.6096) (layer B.Cu) (net 91))
   (segment (start 195.44 109.842) (end 197.612 112.014) (width 0.6096) (layer B.Cu) (net 91))
   (segment (start 195.44 107.808) (end 195.44 109.842) (width 0.6096) (layer B.Cu) (net 91))
-  (segment (start 211.556278 112.014) (end 229.653778 93.9165) (width 0.6096) (layer B.Cu) (net 91))
   (segment (start 304.71364 30.15648) (end 304.74666 30.12346) (width 0.6096) (layer B.Cu) (net 91))
-  (via (at 300.482 93.853) (size 0.8) (drill 0.4) (layers F.Cu B.Cu) (net 91))
-  (segment (start 300.4185 93.9165) (end 300.482 93.853) (width 0.6096) (layer B.Cu) (net 91))
-  (segment (start 229.653778 93.9165) (end 300.4185 93.9165) (width 0.6096) (layer B.Cu) (net 91))
   (via (at 302.514 32.512) (size 0.8) (drill 0.4) (layers F.Cu B.Cu) (net 91))
-  (segment (start 300.482 34.544) (end 302.514 32.512) (width 0.6096) (layer F.Cu) (net 91))
-  (segment (start 300.482 93.853) (end 300.482 34.544) (width 0.6096) (layer F.Cu) (net 91))
   (segment (start 302.514 32.35612) (end 304.74666 30.12346) (width 0.6096) (layer B.Cu) (net 91))
   (segment (start 302.514 32.512) (end 302.514 32.35612) (width 0.6096) (layer B.Cu) (net 91))
+  (segment (start 226.923278 96.647) (end 229.869678 96.647) (width 0.6096) (layer B.Cu) (net 91))
+  (segment (start 211.556278 112.014) (end 226.923278 96.647) (width 0.6096) (layer B.Cu) (net 91))
+  (segment (start 300.482 34.544) (end 300.482 95.7326) (width 0.6096) (layer F.Cu) (net 91))
+  (via (at 299.5676 96.647) (size 0.8) (drill 0.4) (layers F.Cu B.Cu) (net 91))
+  (segment (start 302.514 32.512) (end 300.482 34.544) (width 0.6096) (layer F.Cu) (net 91))
+  (segment (start 300.482 95.7326) (end 299.5676 96.647) (width 0.6096) (layer F.Cu) (net 91))
+  (segment (start 229.869678 96.647) (end 299.5676 96.647) (width 0.6096) (layer B.Cu) (net 91))
   (segment (start 193.04 108.9644) (end 193.04 107.808) (width 0.4064) (layer B.Cu) (net 92))
   (segment (start 193.04 110.035) (end 193.04 108.9644) (width 0.4064) (layer B.Cu) (net 92))

Commit message: Add ESD Protection and make sure the fill zones are on both sides of the board
Parts:
- added U2: USBLC6-2SC6, Package_TO_SOT_SMD:SOT-23-6, B.Cu at (305.5, 27.2)
- moved R2 5.36 mm to (304.4, 32.6)
- moved R3 5.12 mm to (301.6, 32.6)
Routing:
- net USB_VBUS: track 349.8 -> 49.5 mm, vias 8 -> 14
- net GND: track 91.9 -> 81.9 mm, vias 8 -> 2
- net Net-(J1-Pad2): track 5.76 -> 11.5 mm
- net USB_Dneg: track 182.1 -> 176.8 mm
- net USB_Dpos: track 186.8 -> 182.0 mm
- net row3: track 475.7 -> 479.0 mm
- net col15: track 177.9 -> 174.6 mm
- net Net-(J1-Pad3): track 8.32 -> 11.4 mm
- added copper zone on F.Cu, net USB_VBUS

Commit message: Increase the distance between tracks/pads
Routing:
- net row3: track 479.0 -> 321.7 mm
- net row4: track 401.6 -> 488.5 mm
- net GND: track 81.9 -> 93.0 mm, vias 2 -> 5
- net RESET: track 85.7 -> 75.6 mm
- net MOSI: track 255.6 -> 264.0 mm
- net col5: track 171.9 -> 166.1 mm
- net MISO: track 321.9 -> 326.6 mm
- net SCK: track 239.3 -> 243.9 mm
- net col3: track 219.0 -> 215.1 mm
- net col8: track 104.0 -> 101.4 mm
- net col4: track 179.6 -> 177.2 mm
- net row1: track 543.1 -> 540.9 mm
- net col15: track 174.6 -> 176.7 mm
- net row0: track 532.3 -> 534.3 mm
- net col10: track 98.6 -> 100.4 mm
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Other:
- net class Default: clearance 0.127 -> 0.2
- rule trace_clearance: 0.127 -> 0.2
