File: PCB/pcb/_autosave-pcb.kicad_pcb (KiCad board)
At the start: 2 copper layers, 148 parts, among them J1 USB_B_Micro, U1 ATmega32U4-AU, Y1 16MHz

Commit message: New outline (checked with Fusion model)
Other:
- board outline added: 304.8 x 95.2 mm
Changed lines of the file:
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@@
   (general
     (thickness 1.6)
-    (drawings 0)
+    (drawings 10)
     (tracks 0)
     (zones 0)
@@
     )
   )
+  (dimension 304.76825 (width 0.15) (layer Dwgs.User)
+    (gr_text "304.768 mm" (at 169.052875 14.321) (layer Dwgs.User)
+      (effects (font (size 1 1) (thickness 0.15)))
+    )
+    (feature1 (pts (xy 16.66875 19.05) (xy 16.66875 15.034579)))
+    (feature2 (pts (xy 321.437 19.05) (xy 321.437 15.034579)))
+    (crossbar (pts (xy 321.437 15.621) (xy 16.66875 15.621)))
+    (arrow1a (pts (xy 16.66875 15.621) (xy 17.795254 15.034579)))
+    (arrow1b (pts (xy 16.66875 15.621) (xy 17.795254 16.207421)))
+    (arrow2a (pts (xy 321.437 15.621) (xy 320.310496 15.034579)))
+    (arrow2b (pts (xy 321.437 15.621) (xy 320.310496 16.207421)))
+  )
+  (dimension 95.250005 (width 0.15) (layer Dwgs.User)
+    (gr_text "95.250 mm" (at 326.277167 66.673392 270.0190986) (layer Dwgs.User)
+      (effects (font (size 1 1) (thickness 0.15)))
+    )
+    (feature1 (pts (xy 321.46875 114.3) (xy 325.579463 114.29863)))
+    (feature2 (pts (xy 321.437 19.05) (xy 325.547713 19.04863)))
+    (crossbar (pts (xy 324.961292 19.048825) (xy 324.993042 114.298825)))
+    (arrow1a (pts (xy 324.993042 114.298825) (xy 324.406246 113.172517)))
+    (arrow1b (pts (xy 324.993042 114.298825) (xy 325.579087 113.172126)))
+    (arrow2a (pts (xy 324.961292 19.048825) (xy 324.375247 20.175524)))
+    (arrow2b (pts (xy 324.961292 19.048825) (xy 325.548088 20.175133)))
+  )
+  (gr_line (start 16.637 114.3) (end 16.637 19.05) (layer Edge.Cuts) (width 0.05))
+  (gr_line (start 321.437 114.3) (end 16.637 114.3) (layer Edge.Cuts) (width 0.05))
+  (gr_line (start 321.437 19.05) (end 321.437 114.3) (layer Edge.Cuts) (width 0.05))
+  (gr_line (start 16.637 19.05) (end 321.437 19.05) (layer Edge.Cuts) (width 0.05))
+  (target plus (at 16.637 19.05) (size 5) (width 0.05) (layer Edge.Cuts))
+  (target plus (at 16.637 114.3) (size 5) (width 0.05) (layer Edge.Cuts))
+  (target plus (at 321.437 114.3) (size 5) (width 0.05) (layer Edge.Cuts))
+  (target plus (at 321.437 19.05) (size 5) (width 0.05) (layer Edge.Cuts))
 )
