File: PCB/pcb/pcb.sch (KiCad schematic (older format))
At the start: 148 parts, among them J1 USB_B_Micro, U1 ATmega32U4-AU, Y1 16MHz

Commit message: Layout the PCB and generate Gerbers.
I am an idiot. This is my first pass at laying out the board.

What I should have done is mark out the edge cuts and then generate a 3d
model to import into Fusion to check that it fits in the case.

I did not do this until after I'd layed out the board :'( and it's about
5mm too long on each side.

So now I need to make the board smaller by a significant amount and redo
the layout.

Think I learned a lot about laying out a PCB though.
Parts:
- MX1, MX10, MX11, MX12, MX13, MX14, MX15, MX16, MX17, MX18, MX19, MX2, MX20, MX21, MX22, MX23, MX24, MX25, MX26, MX27, MX28, MX29, MX3, MX30, MX31, MX32, MX33, MX34, MX35, MX36, MX37, MX38, MX39, MX4, MX40, MX41, MX42, MX43, MX44, MX45, MX46, MX47, MX48, MX49, MX5, MX50, MX51, MX52, MX53, MX54, MX55, MX56, MX57, MX58, MX59, MX6, MX60, MX61, MX62, MX63, MX64, MX65, MX7, MX8, MX9: symbol pcb-rescue:MX-NoLED-MX_Alps_Hybrid -> MX_Alps_Hybrid:MX-NoLED
Connections:
- net col0: now also U1.11 (PB3); no longer U1.8 (PB0)
- net col1: now also U1.10 (PB2); no longer U1.9 (PB1)
- net col10: now also U1.27 (PD7); no longer U1.32 (PC7)
- net col11: now also U1.28 (PB4); no longer U1.31 (PC6)
- net col12: now also U1.29 (PB5); no longer U1.30 (PB6)
- net col13: now also U1.30 (PB6); no longer U1.29 (PB5)
- net col14: now also U1.31 (PC6); no longer U1.28 (PB4)
- net col15: now also U1.32 (PC7); no longer U1.27 (PD7)
- net col2: now also U1.9 (PB1); no longer U1.10 (PB2)
- net col3: now also U1.8 (PB0); no longer U1.11 (PB3)

Commit message: Finish Layout
Connections:
- net col10: now also U1.28 (PB4); no longer U1.27 (PD7)
- net col11: now also U1.29 (PB5); no longer U1.28 (PB4)
- net col12: now also U1.30 (PB6); no longer U1.29 (PB5)
- net col13: now also U1.31 (PC6); no longer U1.30 (PB6)
- net col14: now also U1.32 (PC7); no longer U1.31 (PC6)
- net col15: now also U1.36 (PF7); no longer U1.32 (PC7)
- net col9: now also U1.27 (PD7); no longer U1.36 (PF7)
Changed lines of the file:
@@
 Text GLabel 4850 5400 1    50   Input ~ 0
 col8
+Text GLabel 3950 5400 1    50   Input ~ 0
+col9
+Text GLabel 2450 5400 1    50   Input ~ 0
+col10
+Text GLabel 2550 5400 1    50   Input ~ 0
+col11
+Text GLabel 2650 5400 1    50   Input ~ 0
+col12
+Text GLabel 2950 5400 1    50   Input ~ 0
+col13
+Text GLabel 3050 5400 1    50   Input ~ 0
+col14
 Text GLabel 4950 5400 1    50   Input ~ 0
-col9
-Text GLabel 3950 5400 1    50   Input ~ 0
-col10
-Text GLabel 2450 5400 1    50   Input ~ 0
-col11
-Text GLabel 2550 5400 1    50   Input ~ 0
-col12
-Text GLabel 2650 5400 1    50   Input ~ 0
-col13
-Text GLabel 2950 5400 1    50   Input ~ 0
-col14
-Text GLabel 3050 5400 1    50   Input ~ 0
 col15
 NoConn ~ 2750 5400
